File: PCB/macropad.kicad_pcb (KiCad board)
At the start: 2 copper layers, 100 x 78 mm, 51 parts, among them J1 Conn_01x04_Pin, SW1 SW_Push_45deg, SW13 RotaryEncoder_Switch, SW14 SW_Push_45deg, SW15 RotaryEncoder_Switch, SW16 SW_Push_45deg, SW17 SW_Push_45deg, SW18 SW_Push_45deg, SW19 SW_Push_45deg, SW2 SW_Push_45deg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

Commit message: Final
Parts:
- moved J1 7.56 mm to (198.0, 36.8), turned to 180 degrees
Connections:
- U1 pad 5: Net-(J1-Pin_3) -> Net-(J1-Pin_4)
- U1 pad 6: Net-(J1-Pin_4) -> Net-(J1-Pin_3)
- U1 pad 7: Net-(D1-VSS) -> unconnected-(U1-GPIO0_D6_TX-Pad7)
Routing:
- net Net-(D1-VSS): track 436.4 -> 409.9 mm, vias 5 -> 6
- net COL1: track 110.5 -> 103.2 mm
- net RE13 B: track 29.7 -> 36.5 mm
- net Net-(D15-DOUT): track 22.3 -> 28.1 mm
- net ROW0: track 86.1 -> 80.7 mm, vias 1 -> 0
- net COL3: track 83.6 -> 78.7 mm
- net Net-(D1-VDD): track 341.4 -> 345.6 mm, vias 9 -> 8
- net Net-(J1-Pin_3): track 13.6 -> 9.98 mm
- net Net-(D1-DIN): track 33.6 -> 30.3 mm
- net COL2: track 129.0 -> 125.8 mm, vias 0 -> 1
- net ROW1: track 100.0 -> 96.9 mm
- net Net-(U1-3V3): track 45.0 -> 47.8 mm
- net Net-(D4-DIN): track 23.1 -> 25.3 mm
- net Net-(D5-DIN): track 78.2 -> 80.2 mm
- net Net-(D3-DIN): track 29.4 -> 30.8 mm
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