File: PCB/macropad.kicad_sch (KiCad schematic)
At the start: 51 parts, among them J1 Conn_01x04_Pin, SW1 SW_Push_45deg, SW13 RotaryEncoder_Switch, SW14 SW_Push_45deg, SW15 RotaryEncoder_Switch, SW16 SW_Push_45deg, SW17 SW_Push_45deg, SW18 SW_Push_45deg, SW19 SW_Push_45deg, SW2 SW_Push_45deg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

Commit message: Final
Connections:
- net at D1.3 (VSS), D10.3 (VSS), D11.3 (VSS)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: no longer U1.7 (GPIO0_D6_TX)
- net at J1.3 (Pin_3): now also U1.6 (GPIO7_D5_SCL); no longer U1.5 (GPIO6_D4_SDA)
- net at J1.4 (Pin_4): now also U1.5 (GPIO6_D4_SDA); no longer U1.6 (GPIO7_D5_SCL)
- no-connect marks 8 -> 9
Changed lines of the file:
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@@
-	)
-	(junction
-		(at 189.23 110.49)
-		(diameter 0)
-		(color 0 0 0 0)
 	)
 	(junction
@@
 		(diameter 0)
 		(color 0 0 0 0)
+	)
+	(no_connect
+		(at 137.16 99.06)
 	)
 	(no_connect
@@
 	(wire
 		(pts
+			(xy 100.33 91.44) (xy 137.16 91.44)
+		)
+		(stroke
+			(width 0)
+			(type default)
+		)
+	)
+	(wire
+		(pts
 			(xy 218.44 151.13) (xy 241.3 151.13)
 		)
@@
 	(wire
 		(pts
-			(xy 100.33 95.25) (xy 100.33 80.01)
+			(xy 100.33 91.44) (xy 100.33 80.01)
 		)
 		(stroke
@@
 	(wire
 		(pts
-			(xy 105.41 91.44) (xy 105.41 77.47)
-		)
-		(stroke
-			(width 0)
-			(type default)
-		)
-	)
-	(wire
-		(pts
-			(xy 189.23 80.01) (xy 189.23 110.49)
+			(xy 105.41 77.47) (xy 105.41 95.25)
 		)
 		(stroke
@@
 	(wire
 		(pts
-			(xy 129.54 99.06) (xy 129.54 110.49)
-		)
-		(stroke
-			(width 0)
-			(type default)
-		)
-	)
-	(wire
-		(pts
 			(xy 189.23 80.01) (xy 191.77 80.01)
 		)
@@
 	(wire
 		(pts
-			(xy 129.54 99.06) (xy 137.16 99.06)
-		)
-		(stroke
-			(width 0)
-			(type default)
-		)
-	)
-	(wire
-		(pts
 			(xy 143.51 38.1) (xy 153.67 38.1)
 		)
@@
 	(wire
 		(pts
+			(xy 105.41 95.25) (xy 137.16 95.25)
+		)
+		(stroke
+			(width 0)
+			(type default)
+		)
+	)
+	(wire
+		(pts
 			(xy 55.88 156.21) (xy 55.88 175.26)
 		)
@@
 	(wire
 		(pts
-			(xy 100.33 95.25) (xy 137.16 95.25)
-		)
-		(stroke
-			(width 0)
-			(type default)
-		)
-	)
-	(wire
-		(pts
 			(xy 191.77 102.87) (xy 204.47 102.87)
 		)
@@
 	(wire
 		(pts
-			(xy 129.54 110.49) (xy 189.23 110.49)
-		)
-		(stroke
-			(width 0)
-			(type default)
-		)
-	)
-	(wire
-		(pts
 			(xy 72.39 168.91) (xy 93.98 168.91)
 		)
@@
 	(wire
 		(pts
-			(xy 189.23 110.49) (xy 189.23 111.76)
+			(xy 189.23 80.01) (xy 189.23 111.76)
 		)
 		(stroke
@@
 		)
 		(stroke
-			(width 0)
-			(type default)
-		)
-	)
-	(wire
-		(pts
-			(xy 105.41 91.44) (xy 137.16 91.44)
-		)
-		(stroke
